File: X3_SOM.sch (KiCad schematic (older format))
At the start: 2 parts

Commit message: file fix
Parts:
- removed U? (x2): X3, symbol otter:X3
- added U? (x3): X3-otter, symbol otter:X3-otter
Connections:
- net +1V1: now also U?.G10 (VDD-CPU), U?.G11 (VDD-CPU), U?.G12 (VDD-CPU), U?.G13 (VDD-CPU), U?.G14 (VDD-CPU), U?.G16 (VDD-SYS), U?.G17 (VDD-SYS), U?.G18 (VDD-SYS), U?.H11 (VDD-CPU), U?.H12 (VDD-CPU), U?.H13 (VDD-CPU), U?.H16 (VDD-SYS), U?.H17 (VDD-SYS), U?.H18 (VDD-SYS), U?.J16 (VDD-SYS), U?.J17 (VDD-SYS), U?.J18 (VDD-SYS), U?.R17 (VCC-CPUS), U?.R18 (VCC-CPUS)
- net +2V5: now also U?.T1 (VDD-DLL), U?.W2 (VCC-EFUSE)
- net +3V0: now also U?.N17 (VCC-IO), U?.N18 (VCC-IO), U?.P17 (VCC-IO), U?.P18 (VCC-IO), U?.X12 (VCC-PD), U?.X26 (VCC-IO), U?.Y12 (VCC-PD), U?.Y26 (VCC-IO)
- net GND: now also U?.A1 (GND), U?.A25 (GND), U?.A26 (GND), U?.B1 (GND), U?.G15 (GND), U?.G9 (GND), U?.H10 (GND), U?.H14 (GND), U?.H15 (GND), U?.H9 (GND), U?.J10 (GND), U?.J11 (GND), U?.J12 (GND), U?.J13 (GND), U?.J14 (GND), U?.J15 (GND), U?.J9 (GND), U?.K10 (GND), U?.K11 (GND), U?.K12 (GND), U?.K13 (GND), U?.K14 (GND), U?.K15 (GND), U?.K16 (GND), U?.K17 (GND), U?.K18 (GND), U?.K9 (GND), U?.L10 (GND), U?.L11 (GND), U?.L12 (GND), U?.L13 (GND), U?.L14 (GND), U?.L15 (GND), U?.L16 (GND), U?.L17 (GND), U?.L18 (GND), U?.L9 (GND), U?.M10 (GND), U?.M11 (GND), U?.M12 (GND), U?.M13 (GND), U?.M14 (GND), U?.M15 (GND), U?.M16 (GND), U?.M17 (GND), U?.M18 (GND), U?.M9 (GND), U?.N10 (GND), U?.N11 (GND), U?.N12 (GND), U?.N13 (GND), U?.N14 (GND), U?.N15 (GND), U?.N16 (GND), U?.N9 (GND), U?.P10 (GND), U?.P14 (GND), U?.P15 (GND), U?.P16 (GND), U?.P9 (GND), U?.R15 (GND), U?.R16 (GND), U?.R9 (GND)
- net GNDA: now also U?.J26 (AGND)
- net VDDA: now also U?.K26 (AVCC)
- new net: U?.P11 (VCC-DRAM), U?.P12 (VCC-DRAM), U?.P13 (VCC-DRAM), U?.R10 (VCC-DRAM), U?.R11 (VCC-DRAM), U?.R12 (VCC-DRAM), U?.R13 (VCC-DRAM), U?.R14 (VCC-DRAM)
- new net: U?.X1 (VCC-DSI), U?.Y1 (VCC-DSI)
Changed lines of the file:
@@
 $EndDescr
-$Comp
-L otter:X3 U?
-U 1 1 5E6BF6A0
-P 2700 4000
-F 0 "U?" H 2700 9165 50  0000 C CNN
-F 1 "X3" H 2700 9074 50  0000 C CNN
-F 2 "" H 1600 2800 50  0001 C CNN
-F 3 "" H 1600 2800 50  0001 C CNN
-	1    2700 4000
-	1    0    0    -1
-$EndComp
-$Comp
-L otter:X3 U?
-U 2 1 5E6C6B04
-P 9900 3850
-F 0 "U?" H 9900 5300 50  0000 C CNN
-F 1 "X3" H 9900 5200 50  0000 C CNN
-F 2 "" H 8800 2650 50  0001 C CNN
-F 3 "" H 8800 2650 50  0001 C CNN
-	2    9900 3850
-	1    0    0    -1
-$EndComp
 $Comp
 L power:+2V5 #PWR?
 U 1 1 5E6D2742
-P 10900 4000
-F 0 "#PWR?" H 10900 3850 50  0001 C CNN
-F 1 "+2V5" V 10915 4128 50  0000 L CNN
-F 2 "" H 10900 4000 50  0001 C CNN
-F 3 "" H 10900 4000 50  0001 C CNN
-	1    10900 4000
+P 11000 4000
+F 0 "#PWR?" H 11000 3850 50  0001 C CNN
+F 1 "+2V5" V 11015 4128 50  0000 L CNN
+F 2 "" H 11000 4000 50  0001 C CNN
+F 3 "" H 11000 4000 50  0001 C CNN
+	1    11000 4000
 	0    1    1    0
 $EndComp
@@
 L power:GNDA #PWR?
 U 1 1 5E6DDAFD
-P 10900 3600
-F 0 "#PWR?" H 10900 3350 50  0001 C CNN
-F 1 "GNDA" V 10905 3472 50  0000 R CNN
-F 2 "" H 10900 3600 50  0001 C CNN
-F 3 "" H 10900 3600 50  0001 C CNN
-	1    10900 3600
+P 11000 3600
+F 0 "#PWR?" H 11000 3350 50  0001 C CNN
+F 1 "GNDA" V 11005 3472 50  0000 R CNN
+F 2 "" H 11000 3600 50  0001 C CNN
+F 3 "" H 11000 3600 50  0001 C CNN
+	1    11000 3600
 	0    -1   -1   0
 $EndComp
@@
 L power:VDDA #PWR?
 U 1 1 5E6DED5A
-P 10900 3400
-F 0 "#PWR?" H 10900 3250 50  0001 C CNN
-F 1 "VDDA" V 10917 3528 50  0000 L CNN
-F 2 "" H 10900 3400 50  0001 C CNN
-F 3 "" H 10900 3400 50  0001 C CNN
-	1    10900 3400
+P 11000 3400
+F 0 "#PWR?" H 11000 3250 50  0001 C CNN
+F 1 "VDDA" V 11017 3528 50  0000 L CNN
+F 2 "" H 11000 3400 50  0001 C CNN
+F 3 "" H 11000 3400 50  0001 C CNN
+	1    11000 3400
 	0    1    1    0
 $EndComp
@@
 L power:+2V5 #PWR?
 U 1 1 5E718BB3
-P 10900 4450
-F 0 "#PWR?" H 10900 4300 50  0001 C CNN
-F 1 "+2V5" V 10915 4578 50  0000 L CNN
-F 2 "" H 10900 4450 50  0001 C CNN
-F 3 "" H 10900 4450 50  0001 C CNN
-	1    10900 4450
+P 11000 4450
+F 0 "#PWR?" H 11000 4300 50  0001 C CNN
+F 1 "+2V5" V 11015 4578 50  0000 L CNN
+F 2 "" H 11000 4450 50  0001 C CNN
+F 3 "" H 11000 4450 50  0001 C CNN
+	1    11000 4450
 	0    1    1    0
 $EndComp
@@
 L power:+3V0 #PWR?
 U 1 1 5E719672
-P 10900 4900
-F 0 "#PWR?" H 10900 4750 50  0001 C CNN
-F 1 "+3V0" V 10915 5028 50  0000 L CNN
-F 2 "" H 10900 4900 50  0001 C CNN
-F 3 "" H 10900 4900 50  0001 C CNN
-	1    10900 4900
+P 11000 4900
+F 0 "#PWR?" H 11000 4750 50  0001 C CNN
+F 1 "+3V0" V 11015 5028 50  0000 L CNN
+F 2 "" H 11000 4900 50  0001 C CNN
+F 3 "" H 11000 4900 50  0001 C CNN
+	1    11000 4900
 	0    1    1    0
 $EndComp
 $Comp
-L power:+3V0 #PWR?
-U 1 1 5E71A923
-P 5800 4900
-F 0 "#PWR?" H 5800 4750 50  0001 C CNN
-F 1 "+3V0" V 5815 5028 50  0000 L CNN
-F 2 "" H 5800 4900 50  0001 C CNN
-F 3 "" H 5800 4900 50  0001 C CNN
-	1    5800 4900
-	0    1    1    0
+L otter:X3-otter U?
+U 1 1 5E6F42E9
+P -3800 2900
+F 0 "U?" H -3800 4815 50  0000 C CNN
+F 1 "X3-otter" H -3800 4724 50  0000 C CNN
+F 2 "" H -3450 4350 50  0001 C CNN
+F 3 "" H -3450 4350 50  0001 C CNN
+	1    -3800 2900
+	1    0    0    -1
 $EndComp
 $Comp
-L power:+1V5 #PWR?
-U 1 1 5E71BD01
-P 5800 5900
-F 0 "#PWR?" H 5800 5750 50  0001 C CNN
-F 1 "+1V5" V 5815 6028 50  0000 L CNN
-F 2 "" H 5800 5900 50  0001 C CNN
-F 3 "" H 5800 5900 50  0001 C CNN
-	1    5800 5900
-	0    1    1    0
+L otter:X3-otter U?
+U 2 1 5E6FC689
+P 550 3200
+F 0 "U?" H 550 5915 50  0000 C CNN
+F 1 "X3-otter" H 550 5824 50  0000 C CNN
+F 2 "" H 900 4650 50  0001 C CNN
+F 3 "" H 900 4650 50  0001 C CNN
+	2    550  3200
+	1    0    0    -1
+$EndComp
+$Comp
+L otter:X3-otter U?
+U 3 1 5E700E89
+P 9900 3850
+F 0 "U?" H 9900 5315 50  0000 C CNN
+F 1 "X3-otter" H 9900 5224 50  0000 C CNN
+F 2 "" H 10250 5300 50  0001 C CNN
+F 3 "" H 10250 5300 50  0001 C CNN
+	3    9900 3850
+	1    0    0    -1
 $EndComp
 $EndSCHEMATC
